Commit message: added dram and slot, pose is wrong, solved shaking issue

File: universal_robot/ur_description/urdf/ur5_ft.urdf.xacro (robot description, xacro)
@@ -350,17 +350,78 @@
       <child link="${prefix}tool0"/>
     </joint>
-  <!-- BEGIN force/torque sensor -->
-  <gazebo reference="wrist_3_joint">
-    <sensor name="wrist_3_joint_force_torque" type="force_torque">
-      <always_on>true</always_on>
-      <update_rate>20.0</update_rate>
-      <visualize>true</visualize>
-      <force_torque>
-        <frame>sensor</frame>
-        <measure_direction>child_to_parent</measure_direction>
-      </force_torque>
-    </sensor>
-  </gazebo>
-  <!-- END force/torque sensor -->
+		<!-- Newly added contents -->
+		<!-- DRAM -->
+		<!-->
+  	<!link name="${prefix}dram">
+  		<visual>
+        <geometry>
+          <mesh filename="package://DRAM_Insert/world/meshes/ram/model.dae" />
+        </geometry>
+      </visual>
+      <collision>
+        <geometry>
+          <mesh filename="package://DRAM_Insert/world/meshes/ram/model.dae" />
+        </geometry>
+      </collision>
+    </link>
+    <joint name="${prefix}tool0-dram_fixed_joint" type="fixed">
+      <origin xyz="0 0 0" rpy="0 0 0"/>
+      <parent link="${prefix}tool0"/>
+      <child link="${prefix}dram"/>
+    </joint>
+    <-->
+		<!-- Gazebo -->
+		<gazebo>
+      <link name='dram'>
+        <pose>1 0.13 0.1 0 1.5707 1.5707</pose>
+        <inertial>
+          <pose>-0.022 0.0203 0.02917 0 0 0</pose>
+          <mass>0.00001</mass>
+          <inertia>
+            <ixx>0.00001</ixx>
+            <ixy>0</ixy>
+            <ixz>0</ixz>
+            <iyy>0.00001</iyy>
+            <iyz>0</iyz>
+            <izz>0.00001</izz>
+          </inertia>
+        </inertial>
+        <collision name='dram_collision'>
+          <geometry>
+            <mesh>
+              <!-- Load a local mesh model. https://answers.gazebosim.org//question/6568/uri-paths-to-packages-in-the-sdf-model-file/ -->
+              <uri>model://DRAM_Insert/world/meshes/ram/model.dae</uri>
+              <!--scale>1 1 1</scale-->
+              </mesh>
+          </geometry>
+        </collision>
+        <visual name='dram_visual'>
+          <!--pose>0 0 0 0 1.5707 1.5707</pose-->
+          <geometry>
+            <mesh>
+              <!-- Load a local mesh model. https://answers.gazebosim.org//question/6568/uri-paths-to-packages-in-the-sdf-model-file/ -->
+              <uri>model://DRAM_Insert/world/meshes/ram/model.dae</uri>
+              <!--scale>1 1 1</scale-->
+            </mesh>
+          </geometry>
+        </visual>
+      </link>
+      <joint name='dram_joint' type='fixed'>
+        <child>dram</child>
+        <parent>wrist_3_link</parent>
+      </joint>
+    </gazebo>
+		<!-- Force/torque sensor -->
+		<gazebo reference="wrist_3_joint"> <!-- http://gazebosim.org/tutorials/?tut=ros_urdf -->
+		  <sensor name="wrist_3_joint_force_torque" type="force_torque">
+		    <always_on>true</always_on>
+		    <update_rate>20.0</update_rate>
+		    <visualize>true</visualize>
+		    <force_torque>
+		      <frame>sensor</frame>  <!-- https://gazebosim.org/tutorials?tut=force_torque_sensor&cat=sensors -->
+		      <measure_direction>child_to_parent</measure_direction>
+		    </force_torque>
+		  </sensor>
+		</gazebo>
   </xacro:macro>
 </robot>
